File: hardware/CH32X035_XIAO-Compatible_Board/CH32X035_XIAO-Compatible_Board.kicad_pcb (KiCad board)
At the start: 4 copper layers, 17.8 x 21 mm, 20 parts, among them IC1 TCR1HF33B, J1 GCT USB4105, J2 Conn_01x07, J3 Conn_01x07, J4 Conn_02x05_Odd_Even, SW1 SW_Push, U3 CH32X035C8T6

Commit message: サポートページ用の回路図・基板設計データの変更
Other:
- board text added: "CH32 X035 C8T6"
- board text added: "VBUS =PA4x11"
- board text added: "XIAO COMPATIBLE"
- board text removed: "XIAO CH32X035"
Changed lines of the file:
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@@
   (paper "A4")
   (title_block
-    (title "XIAO_CH32X035")
-    (date "2024-06-27")
-    (rev "v1.0")
+    (title "CH32X035 XIAO-Compatible Board")
+    (date "2024-09-02")
+    (rev "v2.0")
     (company "@suzan_works")
   )
@@
   (gr_rect (start 115.88 79.05) (end 117.78 80.95)
     (stroke (width 0.001) (type default)) (fill none) (layer "User.2"))
-  (gr_text "XIAO CH32X035" (at 114.7 82.6) (layer "B.SilkS")
+  (gr_text "XIAO COMPATIBLE" (at 114.9 82.6) (layer "B.SilkS")
     (effects (font (size 0.9 0.9) (thickness 0.15)) (justify left bottom mirror))
   )
-  (gr_text "JP TO USB" (at 112.4 86.7) (layer "B.SilkS")
+  (gr_text "JP TO USB" (at 112.4 86.6) (layer "B.SilkS")
+    (effects (font (size 0.8 0.8) (thickness 0.15)) (justify left bottom mirror))
+  )
+  (gr_text "CH32\nX035\nC8T6" (at 115.3 90.55) (layer "B.SilkS")
     (effects (font (size 0.8 0.8) (thickness 0.15)) (justify left bottom mirror))
   )
@@
     (effects (font (size 0.9 0.9) (thickness 0.15)) (justify left bottom))
   )
-  (gr_text "XIAO\nCH32X035" (at 109.1 88.3) (layer "F.SilkS")
-    (effects (font (size 0.9 0.9) (thickness 0.15)) (justify bottom))
+  (gr_text "VBUS\n=PA4x11" (at 105.8 88.35) (layer "F.SilkS")
+    (effects (font (size 0.9 0.9) (thickness 0.15)) (justify left bottom))
   )
   (gr_text "TX" (at 102.1 96.5 270) (layer "F.SilkS")
