File: hardware/CH32X035_XIAO-Compatible_Board/CH32X035_XIAO-Compatible_Board.kicad_sch (KiCad schematic)
At the start: 20 parts, among them IC1 TCR1HF33B, J1 GCT USB4105, J2 2.54mm Pin Header, J3 Conn_01x07, J4 1.27mm 2x5P, SW1 SW_Push, U3 CH32X035C8T6

Commit message: サポートページ用の回路図・基板設計データの変更
Parts:
- F1: value 0603L010YR -> MF-FSMF010X
Other:
- title: XIAO_CH32X035 -> CH32X035 XIAO-Compatible Board
Changed lines of the file:
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@@
   (paper "A4")
   (title_block
-    (title "XIAO_CH32X035")
-    (date "2024-06-25")
-    (rev "v1.0")
+    (title "CH32X035 XIAO-Compatible Board")
+    (date "2024-09-02")
+    (rev "v2.0")
     (company "@suzan_works")
   )
