File: hardware/SWD_Converter_Board/SWD_Converter_Board.kicad_pcb (KiCad board)
At the start: 2 copper layers, 17.8 x 39.4 mm, 5 parts, among them J1 Conn_02x05_Odd_Even, J2 Conn_02x05_Odd_Even, J3 Conn_01x05, J4 Conn_01x05, SW1 SW_SPDT

Commit message: サポートページ用の回路図・基板設計データの変更
Routing:
- net /RST: track 30.9 -> 32.0 mm
Other:
- board text added: "3V3 OUTPUT"
- board text added: "SWD CONVERTER"
- board text removed: "3V3 OUT SW"
- board text removed: "WCH-LinkE Converter"
