File: hardware/SWD_Converter_Board/SWD_Converter_Board.kicad_sch (KiCad schematic)
At the start: 5 parts, among them J1 2.54mm 2x5P, J2 1.27mm 2x5P, J3 2.54mm, J4 Conn_01x05, SW1 SW_SPDT

Commit message: サポートページ用の回路図・基板設計データの変更
Other:
- title: WCH-LinkE_adapter -> SWD Converter Board
Changed lines of the file:
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@@
   (paper "A4")
   (title_block
-    (title "WCH-LinkE_adapter")
-    (date "2024-06-25")
-    (rev "v1.0")
+    (title "SWD Converter Board")
+    (date "2024-09-02")
+    (rev "v2.0")
     (company "@suzan_works")
   )
@@
     (pin "9")
     (instances
-      (project "WCHLinkE_Converter_2"
+      (project "WCHLinkE_Converter_5"
         (path "/575a9c30-2b78-4eea-a8f3-c2ee267e357b"
           (reference "J2") (unit 1)
@@
     (pin "3")
     (instances
-      (project "WCHLinkE_Converter_2"
+      (project "WCHLinkE_Converter_5"
         (path "/575a9c30-2b78-4eea-a8f3-c2ee267e357b"
           (reference "SW1") (unit 1)
@@
     (pin "9")
     (instances
-      (project "WCHLinkE_Converter_2"
+      (project "WCHLinkE_Converter_5"
         (path "/575a9c30-2b78-4eea-a8f3-c2ee267e357b"
           (reference "J1") (unit 1)
@@
     (pin "5")
     (instances
-      (project "WCHLinkE_Converter_2"
+      (project "WCHLinkE_Converter_5"
         (path "/575a9c30-2b78-4eea-a8f3-c2ee267e357b"
           (reference "J3") (unit 1)
@@
     (pin "5")
     (instances
-      (project "WCHLinkE_Converter_2"
+      (project "WCHLinkE_Converter_5"
         (path "/575a9c30-2b78-4eea-a8f3-c2ee267e357b"
           (reference "J4") (unit 1)
