File: hardware/VBUS_Switch_Addon_Board/VBUS_Switch_Addon_Board.kicad_sch (KiCad schematic)
At the start: 15 parts, among them IC1 TCR1HF50B, IC2 FDS4935A, IC3 ACS724LLCTR-05AB, J1 2.54mm Pin Header, J2 Conn_01x07, J3 2.54mm Screw Terminal, Q1 DTC143Z, SW1 SW_Push, SW2 SW_Push

Commit message: サポートページ用の回路図・基板設計データの変更
Parts:
- added D1: Red LED, LED_SMD:LED_0402_1005Metric, symbol Device:LED
- added J4, J5: 1.3mm Through Hole, Connector_Pin:Pin_D1.3mm_L11.0mm, symbol Connector_Generic:Conn_01x01
- added JP1: SolderJumper_2_Open, 0_My_Library:SolderJumper-2_P1.3mm_Open_Pad0.8x1.2mm, symbol Jumper:SolderJumper_2_Open
- added R3: 220, Resistor_SMD:R_0402_1005Metric, symbol Device:R_Small
- added R4, R5: 10k, Resistor_SMD:R_0402_1005Metric, symbol Device:R_Small
- J3: value 2.54mm Screw Terminal -> Terminal Block
Connections:
- net +5V: now also JP1.2 (B)
- net GND: now also D1.1 (K), J5.1 (Pin_1), R5.2
- net PA0: now also R3.1
- net PA1: now also R4.2, R5.1; no longer IC3.7 (VIOUT)
- net VBUS: now also JP1.1 (A)
- net at IC3.3 (IP-_1), IC3.4 (IP-_2), J3.1 (Pin_1): now also J4.1 (Pin_1)
- new net: IC3.7 (VIOUT), R4.1
- new net: D1.2 (A), R3.2
Other:
- note added: "Output Indicator LED"
- note added: "Short JP1 only when VBUS = 5V."
- note removed: "・出力インジケータLEDを追加予定です。 ・電流センサーICの出力に抵抗を追加予定です。分圧してからPA1に入力します。 ・5Vレギュレータ用にVBUS5V時の切替スイッチを追加予定です。 - Add output LED. - Add resistors to current sensor output for division into PA1. - Add switch for 5V regulator."
- title: VBUS_SWITCH_BFF -> VBUS Switch Addon Board
